File: PowerManagementMysensors/PowerManagementMysensors.brd (EAGLE design)
At the start: 49.5 x 44.1 mm, 52 parts, among them IC2 AT25DF512C-SSHN-B, U1 LM8364BALMF20, U2 SI2399DS-T1-GE3, U3 SI2399DS-T1-GE3, U4 MCP1640BT-I/CHY, U5 TPS61222DCKT

Commit message: silkscreen changed, Bom added
Parts:
- L1, L2: device SparkFun-Passives:1210 -> SparkFun-Passives:0805
Routing:
- net N$13: track 10.0 -> 10.6 mm
- net N$10: track 4.14 -> 4.73 mm
Changed lines of the file:
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@@
 <layer number="20" name="Dimension" color="15" fill="1" visible="yes" active="yes"/>
 <layer number="21" name="tPlace" color="7" fill="1" visible="yes" active="yes"/>
-<layer number="22" name="bPlace" color="7" fill="1" visible="no" active="yes"/>
+<layer number="22" name="bPlace" color="7" fill="1" visible="yes" active="yes"/>
 <layer number="23" name="tOrigins" color="15" fill="1" visible="no" active="yes"/>
 <layer number="24" name="bOrigins" color="15" fill="1" visible="no" active="yes"/>
@@
 <attribute name="VALUE" x="32.9057" y="-1.1684" size="2.0828" layer="28" ratio="10" rot="SMR90"/>
 </element>
-<element name="L1" library="SparkFun-Passives" package="1210" value="4.7uH" x="43.3451" y="4.1529" smashed="yes" rot="MR270">
+<element name="L1" library="SparkFun-Passives" package="0805" value="4.7uH" x="43.3451" y="4.1529" smashed="yes" rot="MR270">
 <attribute name="NAME" x="45.4105" y="4.0131" size="0.4064" layer="26" rot="MR270"/>
 <attribute name="VALUE" x="44.0451" y="5.0529" size="0.4064" layer="28" rot="MR270"/>
@@
 <element name="R4" library="SparkFun-Passives" package="1206" value="470k" x="33.02" y="31.115" rot="MR0"/>
 <element name="APM" library="pmo_lib" package="ARDUINO_PROMINI2" value="ARDUINO_PROMINI2" x="17.78" y="34.29" smashed="yes" rot="R270">
-<attribute name="NAME" x="19.05" y="36.83" size="1.27" layer="25"/>
+<attribute name="NAME" x="11.2014" y="36.6268" size="1.27" layer="25"/>
 <attribute name="VALUE" x="0" y="36.83" size="1.27" layer="27" rot="R270"/>
 </element>
@@
 <attribute name="VALUE" x="50.4825" y="13.6144" size="2.0828" layer="28" ratio="10" rot="SMR270"/>
 </element>
-<element name="L2" library="SparkFun-Passives" package="1210" value="4.7uH" x="43.2435" y="10.16" smashed="yes" rot="MR270">
+<element name="L2" library="SparkFun-Passives" package="0805" value="4.7uH" x="43.2435" y="10.16" smashed="yes" rot="MR270">
 <attribute name="NAME" x="41.6513" y="10.4012" size="0.4064" layer="26" rot="MR270"/>
 <attribute name="VALUE" x="43.9435" y="11.06" size="0.4064" layer="28" rot="MR270"/>
@@
 <contactref element="L1" pad="2"/>
 <contactref element="U4" pad="1"/>
-<wire x1="43.3451" y1="2.5529" x2="38.7094" y2="2.5275" width="0.4064" layer="16"/>
-<wire x1="38.7094" y1="2.5275" x2="38.0873" y2="3.1496" width="0.4064" layer="16"/>
+<wire x1="38.0873" y1="3.1496" x2="38.1508" y2="3.1496" width="0.6096" layer="16"/>
+<wire x1="38.1508" y1="3.1496" x2="38.989" y2="2.3114" width="0.6096" layer="16"/>
+<wire x1="38.989" y1="2.3114" x2="42.4036" y2="2.3114" width="0.6096" layer="16"/>
+<wire x1="42.4036" y1="2.3114" x2="43.3451" y2="3.2529" width="0.6096" layer="16"/>
 </signal>
 <signal name="N$4">
@@
 <wire x1="46.0375" y1="9.1186" x2="46.0375" y2="8.1915" width="0.6096" layer="16"/>
 <wire x1="46.0375" y1="8.1915" x2="45.72" y2="7.874" width="0.6096" layer="16"/>
-<wire x1="45.72" y1="7.874" x2="43.9295" y2="7.874" width="0.6096" layer="16"/>
-<wire x1="43.9295" y1="7.874" x2="43.2435" y2="8.56" width="0.6096" layer="16"/>
+<wire x1="45.72" y1="7.874" x2="44.196" y2="7.874" width="0.6096" layer="16"/>
+<wire x1="44.196" y1="7.874" x2="43.18" y2="8.89" width="0.6096" layer="16"/>
+<wire x1="43.18" y1="8.89" x2="43.18" y2="9.1965" width="0.6096" layer="16"/>
+<wire x1="43.18" y1="9.1965" x2="43.2435" y2="9.26" width="0.6096" layer="16"/>
 </signal>
 <signal name="V+5">
@@
 <contactref element="JP3" pad="1"/>
 <wire x1="45.3771" y1="11.2014" x2="45.3771" y2="9.1186" width="0.4064" layer="16"/>
-<wire x1="43.31" y1="11.8265" x2="43.2435" y2="11.76" width="0.4064" layer="16"/>
 <wire x1="43.31" y1="15.8175" x2="43.3675" y2="15.875" width="0.4064" layer="16"/>
-<wire x1="43.31" y1="11.8265" x2="43.31" y2="11.935" width="0.4064" layer="16"/>
-<wire x1="43.31" y1="11.935" x2="43.2465" y2="11.935" width="0.4064" layer="16"/>
-<wire x1="43.2465" y1="11.935" x2="40.386" y2="14.7955" width="0.8128" layer="16"/>
 <wire x1="40.386" y1="14.7955" x2="40.386" y2="14.986" width="0.8128" layer="16"/>
 <wire x1="40.386" y1="14.986" x2="41.275" y2="15.875" width="0.8128" layer="16"/>
@@
 <polygon width="0.254" layer="16">
 <vertex x="41.91" y="12.065"/>
-<vertex x="41.91" y="10.16"/>
-<vertex x="45.339" y="10.16"/>
+<vertex x="41.8846" y="10.4648"/>
+<vertex x="45.3136" y="10.4648"/>
 <vertex x="45.339" y="12.065"/>
 </polygon>
+<wire x1="40.386" y1="14.7955" x2="40.386" y2="14.7066" width="0.8128" layer="16"/>
+<wire x1="40.386" y1="14.7066" x2="43.1292" y2="11.9634" width="0.8128" layer="16"/>
+<wire x1="43.1292" y1="11.9634" x2="43.1292" y2="11.1743" width="0.8128" layer="16"/>
+<wire x1="43.1292" y1="11.1743" x2="43.2435" y2="11.06" width="0.8128" layer="16"/>
 </signal>
 <signal name="N$8">
@@
 <vertex x="39.0144" y="5.6388"/>
 <vertex x="41.91" y="5.6388"/>
-<vertex x="41.91" y="4.2672"/>
-<vertex x="44.8056" y="4.2926"/>
+<vertex x="41.91" y="4.445"/>
+<vertex x="44.8056" y="4.4704"/>
 <vertex x="44.7802" y="6.4008"/>
-<vertex x="44.7548" y="7.1628"/>
+<vertex x="43.8658" y="6.5532"/>
 <vertex x="41.0972" y="7.1628"/>
 <vertex x="40.64" y="7.62"/>
