File: PowerManagementMysensors/PowerManagementMysensors2.brd (EAGLE design)
At the start: 49.5 x 44.1 mm, 52 parts, among them IC2 AT25DF512C-SSHN-B, U1 LM8364BALMF20, U2 SI2399DS-T1-GE3, U3 SI2399DS-T1-GE3, U4 MCP1640BT-I/CHY, U5 TPS61222DCKT

Commit message: silkscreen changed, Bom added
Parts:
- L1, L2: device SparkFun-Passives:1210 -> SparkFun-Passives:0805
Routing:
- net N$1: track 5.52 -> 6.23 mm
- net N$13: track 10.0 -> 10.6 mm
- net N$10: track 4.14 -> 4.73 mm
Changed lines of the file:
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@@
 <attribute name="VALUE" x="32.9057" y="-1.1684" size="2.0828" layer="28" ratio="10" rot="SMR90"/>
 </element>
-<element name="L1" library="SparkFun-Passives" package="1210" value="4.7uH" x="43.3451" y="4.1529" smashed="yes" rot="MR270">
+<element name="L1" library="SparkFun-Passives" package="0805" value="4.7uH" x="43.3451" y="4.1529" smashed="yes" rot="MR270">
 <attribute name="NAME" x="45.4105" y="4.0131" size="0.4064" layer="26" rot="MR270"/>
 <attribute name="VALUE" x="44.0451" y="5.0529" size="0.4064" layer="28" rot="MR270"/>
@@
 <attribute name="VALUE" x="50.4825" y="13.6144" size="2.0828" layer="28" ratio="10" rot="SMR270"/>
 </element>
-<element name="L2" library="SparkFun-Passives" package="1210" value="4.7uH" x="43.2435" y="10.16" smashed="yes" rot="MR270">
+<element name="L2" library="SparkFun-Passives" package="0805" value="4.7uH" x="43.2435" y="10.16" smashed="yes" rot="MR270">
 <attribute name="NAME" x="41.6513" y="10.4012" size="0.4064" layer="26" rot="MR270"/>
 <attribute name="VALUE" x="43.9435" y="11.06" size="0.4064" layer="28" rot="MR270"/>
@@
 <contactref element="L1" pad="2"/>
 <contactref element="U4" pad="1"/>
-<wire x1="43.3451" y1="2.5529" x2="38.7094" y2="2.5275" width="0.4064" layer="16"/>
-<wire x1="38.7094" y1="2.5275" x2="38.0873" y2="3.1496" width="0.4064" layer="16"/>
+<wire x1="38.0873" y1="3.1496" x2="38.0873" y2="2.8575" width="0.6096" layer="16"/>
+<wire x1="38.0873" y1="2.8575" x2="38.7096" y2="2.2352" width="0.6096" layer="16"/>
+<wire x1="38.7096" y1="2.2352" x2="42.3274" y2="2.2352" width="0.6096" layer="16"/>
+<wire x1="42.3274" y1="2.2352" x2="43.3451" y2="3.2529" width="0.6096" layer="16"/>
 </signal>
 <signal name="N$4">
@@
 <wire x1="46.0375" y1="9.1186" x2="46.0375" y2="8.1915" width="0.6096" layer="16"/>
 <wire x1="46.0375" y1="8.1915" x2="45.72" y2="7.874" width="0.6096" layer="16"/>
-<wire x1="45.72" y1="7.874" x2="43.9295" y2="7.874" width="0.6096" layer="16"/>
-<wire x1="43.9295" y1="7.874" x2="43.2435" y2="8.56" width="0.6096" layer="16"/>
+<wire x1="45.72" y1="7.874" x2="44.196" y2="7.874" width="0.6096" layer="16"/>
+<wire x1="44.196" y1="7.874" x2="43.18" y2="8.89" width="0.6096" layer="16"/>
+<wire x1="43.18" y1="8.89" x2="43.18" y2="9.1965" width="0.6096" layer="16"/>
+<wire x1="43.18" y1="9.1965" x2="43.2435" y2="9.26" width="0.6096" layer="16"/>
 </signal>
 <signal name="V+5">
@@
 <contactref element="JP3" pad="1"/>
 <wire x1="45.3771" y1="11.2014" x2="45.3771" y2="9.1186" width="0.4064" layer="16"/>
-<wire x1="43.31" y1="11.8265" x2="43.2435" y2="11.76" width="0.4064" layer="16"/>
 <wire x1="43.31" y1="15.8175" x2="43.3675" y2="15.875" width="0.4064" layer="16"/>
-<wire x1="43.31" y1="11.8265" x2="43.31" y2="11.935" width="0.4064" layer="16"/>
-<wire x1="43.31" y1="11.935" x2="43.2465" y2="11.935" width="0.4064" layer="16"/>
-<wire x1="43.2465" y1="11.935" x2="40.386" y2="14.7955" width="0.8128" layer="16"/>
 <wire x1="40.386" y1="14.7955" x2="40.386" y2="14.986" width="0.8128" layer="16"/>
 <wire x1="40.386" y1="14.986" x2="41.275" y2="15.875" width="0.8128" layer="16"/>
@@
 <polygon width="0.254" layer="16">
 <vertex x="41.91" y="12.065"/>
-<vertex x="41.91" y="10.16"/>
-<vertex x="45.339" y="10.16"/>
+<vertex x="41.9354" y="10.541"/>
+<vertex x="45.3644" y="10.541"/>
 <vertex x="45.339" y="12.065"/>
 </polygon>
+<wire x1="40.386" y1="14.7955" x2="40.386" y2="14.6812" width="0.8128" layer="16"/>
+<wire x1="40.386" y1="14.6812" x2="43.2054" y2="11.8618" width="0.8128" layer="16"/>
+<wire x1="43.2054" y1="11.8618" x2="43.2054" y2="11.0981" width="0.8128" layer="16"/>
+<wire x1="43.2054" y1="11.0981" x2="43.2435" y2="11.06" width="0.8128" layer="16"/>
 </signal>
 <signal name="N$8">
@@
 <vertex x="44.8056" y="4.2926"/>
 <vertex x="44.7802" y="6.4008"/>
-<vertex x="44.7548" y="7.1628"/>
+<vertex x="43.2562" y="6.731"/>
 <vertex x="41.0972" y="7.1628"/>
 <vertex x="40.64" y="7.62"/>
