File: OneRelayMysensors/OneRelayMysensors.brd (EAGLE design)
At the start: 38.2 x 43.2 mm, 33 parts, among them IC1 MEGA328P-AU, Q1 32768hz, T1 BC847BW-7-F

Commit message: relay footprint, changes res size
Parts:
- added P1, P2, P3: (no value), wirepad:2,54/1,1
- R4, R5: device Discrete:R0805 -> SparkFun-Passives:1206
- moved R5 0.96 mm to (20.0, 21.9), turned to 225 degrees
- moved R4 0.90 mm to (27.3, 27.3), turned to 0 degrees
Connections:
- net REL2B: now also P3.1
- net REL4: now also P1.1
- net REL5: now also P2.1
Routing:
- net RST: track 37.7 -> 36.2 mm
- net A2: track 3.42 -> 4.00 mm
- net REL5: track 5.96 -> 5.87 mm, vias 1 -> 0
- net REL4: track 5.96 -> 5.87 mm, vias 1 -> 0
- net REL2B: vias 1 -> 0
