File: RollerShutterNode/nrf24_smd/RollerShutterNode_nrf_1-1_EN.sch (EAGLE design)
At the start: 50 parts, among them IC1 ATMega-328, IC2 AT25DF512C-SSHN-B, IC3 MCP1703CB, IC4 ACS712_5A, IC5 ATSHA204A, IC6 LM321, IC7 MDC3105DMT1, X1 8 MHz

Commit message: 1.1 update
there was a missing mistake I didn't see even if I checked lot of
times...routing derouting mistake...spst relay was always ON. shame on
me!
Connections:
- new net TOGGLE: IC4.IP+, IC4.IP+_2, RL1.NC
- net 12_220: no longer IC4.IP+, IC4.IP+_2
- net COM: no longer RL1.NC
Changed lines of the file:
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@@
 </segment>
 <segment>
-<wire x1="144.78" y1="78.74" x2="144.78" y2="93.98" width="0.1524" layer="91"/>
 <pinref part="RL2" gate="G$1" pin="MAIN"/>
 <wire x1="144.78" y1="93.98" x2="127" y2="93.98" width="0.1524" layer="91"/>
-<label x="144.78" y="78.74" size="1.778" layer="95" xref="yes"/>
-<pinref part="RL1" gate="G$1" pin="NC"/>
-<wire x1="139.7" y1="78.74" x2="144.78" y2="78.74" width="0.1524" layer="91"/>
+<label x="144.78" y="93.98" size="1.778" layer="95" xref="yes"/>
 </segment>
 </net>
@@
 <wire x1="177.8" y1="86.36" x2="175.26" y2="88.9" width="0.1524" layer="91"/>
 <label x="175.26" y="88.9" size="1.778" layer="95" rot="R180" xref="yes"/>
-</segment>
-<segment>
-<label x="205.74" y="53.34" size="1.778" layer="95" rot="R180" xref="yes"/>
-<pinref part="IC4" gate="A" pin="IP+_2"/>
-<wire x1="215.9" y1="53.34" x2="205.74" y2="53.34" width="0.1524" layer="91"/>
-<wire x1="220.98" y1="60.96" x2="215.9" y2="60.96" width="0.1524" layer="91"/>
-<wire x1="215.9" y1="60.96" x2="215.9" y2="55.88" width="0.1524" layer="91"/>
-<pinref part="IC4" gate="A" pin="IP+"/>
-<wire x1="215.9" y1="55.88" x2="220.98" y2="55.88" width="0.1524" layer="91"/>
-<wire x1="215.9" y1="55.88" x2="215.9" y2="53.34" width="0.1524" layer="91"/>
-<junction x="215.9" y="55.88"/>
 </segment>
 <segment>
@@
 </segment>
 </net>
+<net name="TOGGLE" class="0">
+<segment>
+<label x="205.74" y="53.34" size="1.778" layer="95" rot="R180" xref="yes"/>
+<pinref part="IC4" gate="A" pin="IP+_2"/>
+<wire x1="215.9" y1="53.34" x2="205.74" y2="53.34" width="0.1524" layer="91"/>
+<wire x1="220.98" y1="60.96" x2="215.9" y2="60.96" width="0.1524" layer="91"/>
+<wire x1="215.9" y1="60.96" x2="215.9" y2="55.88" width="0.1524" layer="91"/>
+<pinref part="IC4" gate="A" pin="IP+"/>
+<wire x1="215.9" y1="55.88" x2="220.98" y2="55.88" width="0.1524" layer="91"/>
+<wire x1="215.9" y1="55.88" x2="215.9" y2="53.34" width="0.1524" layer="91"/>
+<junction x="215.9" y="55.88"/>
+</segment>
+<segment>
+<pinref part="RL1" gate="G$1" pin="NC"/>
+<wire x1="139.7" y1="78.74" x2="144.78" y2="78.74" width="0.1524" layer="91"/>
+<label x="144.78" y="78.74" size="1.778" layer="95" xref="yes"/>
+</segment>
+</net>
