File: RollerShutterNode/rfm69/MyRollerShutter_rfm.sch (EAGLE design)
At the start: 52 parts, among them IC1 ATMega-328, IC2 AT25DF512C-SSHN-B, IC3 MCP1703CB, IC4 ACS712_5A, IC5 ATSHA204A, IC6 LM321, U1 MDC3105DMT1, X1 8 MHz

Commit message: some rerouting and a small fix on connector
Parts:
- removed M: (no value), SparkFun-Connectors:M03-SCREW-5MM
- added MOTOR: (no value), SparkFun-Connectors:M03-SCREW-5MM
Connections:
- net COM renamed OUT_ACS
- net NEUTRE renamed N
- net TOGGLE renamed IN_ACS
- net 12_220: now also MOTOR.3; no longer M.3
- net L: no longer AC.1
- net M_DOWN: now also MOTOR.1; no longer M.1
- net M_UP: now also MOTOR.2; no longer M.2
- net PHASE: now also AC.1
Other:
- note added: "Atmel decoupling"
- note added: "Current sensor"
- note added: "For 110/220V motor : connect 12_220 to PHASE For 12V/24V motor : connect 12_220 to your 12/24V source"
- note added: "Input protection : Varistor + 5A fuse"
- note added: "Monitoring board temperature"
- note added: "Motor connection : - Neutral to N - UP to M_UP - DOWN to M_DOWN"
- note added: "Note :there is no snubber. external if needed"
- note added: "Power input & Protection : 110-220V -> 5V and+ 3.3V Reg"
- note added: "Radio"
- note added: "Relays"
- note added: "SMD PINHEADER 1) AVRSPI 2) Buttons - Up - Down - Stop 3) I2C SDA/SCL : - for i2c control chip : tactile, gesture.. - D3 : option i/o, interrupt, for i2c chip... - D4 : option i/o"
- note added: "Upload and authentication"
- note added: "low pass RC filter for acs712, Optional"
- note removed: "Alimentation et protection : 220V -> 5V, Régulateur 3V"
- note removed: "Analyse courant"
- note removed: "Découplage Atmel"
- note removed: "Filtre en sortie"
- note removed: "Module RF"
- note removed: "Monitoring température board"
- note removed: "Note : il n'y a pas de snubber. Si nécessaire le mettre en externe"
- note removed: "Pilotage relais"
- note removed: "Pour acs712, filtre RC low pass Optionnel"
- note removed: "Protection en entrée : Varistance + fusible 5A"
- note removed: "SMD PINHEADER 1) Boutons DC - Bouton Up : Monter volet - Bouton Down : Descendre volet - Bouton Stop : Stopper le moteur 2) I2C externe - possibilité de connecter une interface externe de pilotage - D3, D4 au cas où l'extension nécessite des broches supp."
- note removed: "Upload et sécurité"
- moved on the sheet: AC, C1, C10, C11, C12, C15, C2, C3, C6, D3, F1, FTDI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
