File: RollerShutterNode/Eagle/NRF24_SMD/MyRollerShutter_nrf_1-3a.brd (EAGLE design)
At the start: 44.4 x 45.4 mm, 64 parts, among them IC1 ATMega-328, IC2 AT25DF512C-SSHN-B, IC3 MCP1703CB, IC4 ACS712_5A, IC5 ATSHA204A, IC6 LM321, IC7 MDC3105DMT1, IC8 DS1820, J1 SCREW-TERMINAL-2P-3470110P1, J2 SCREW-TERMINAL-2P-3470110P1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

Commit message: nrf24 minor fix
CSN was not connected in pcb! whereas it was in schematics..
Connections:
- removed net N$8: NRF_SMD.CSN
- net RF_CSN: now also NRF_SMD.CSN
Routing:
- net RF_CSN: track 22.5 -> 25.0 mm
Other:
- board text added: "RollersShutterNode r1.3a (c) Scalz 2016"
- board text removed: "Creepage sample"
- board text removed: "RollersShutterNode r1.3 (c) Scalz 2016 rev 1.3"
Changed lines of the file:
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@@
 <wire x1="42.525" y1="0" x2="44.43" y2="1.905" width="0" layer="20" curve="90"/>
 <text x="42.7736" y="16.3576" size="0.8128" layer="22" rot="MR0">HIGH VOLTAGE SIDE. Be careful. Risk of death!</text>
-<text x="0.762" y="42.5196" size="0.6096" layer="21" font="vector">RollersShutterNode r1.3
-(c) Scalz 2016 rev 1.3</text>
+<text x="0.762" y="42.5196" size="0.6096" layer="21" font="vector">RollersShutterNode r1.3a
+(c) Scalz 2016</text>
 <text x="41.783" y="0.635" size="0.8128" layer="22" font="vector" rot="MR0">N</text>
 <text x="36.322" y="0.635" size="0.8128" layer="22" font="vector" rot="MR0">L</text>
@@
 <text x="9.2456" y="0.508" size="0.8128" layer="22" font="vector" rot="MR0">UP</text>
 <text x="4.8006" y="0.508" size="0.8128" layer="22" font="vector" rot="MR0">DOWN</text>
-<wire x1="-1.06860625" y1="15.630025" x2="-1.06860625" y2="12.76536875" width="0.254" layer="51"/>
 <wire x1="6.096" y1="2.032" x2="6.096" y2="12.192" width="1.27" layer="46"/>
 <wire x1="17.907" y1="2.032" x2="17.907" y2="11.176" width="1.27" layer="46"/>
@@
 <wire x1="11.684" y1="2.032" x2="11.684" y2="14.224" width="1.27" layer="46"/>
 <wire x1="34.036" y1="14.732" x2="20.828" y2="14.732" width="1.27" layer="46"/>
-<dimension x1="-1.06860625" y1="15.630025" x2="-1.06860625" y2="12.76536875" x3="-2.54" y3="14.197696875" textsize="1.778" layer="51"/>
-<dimension x1="1.905" y1="45.39" x2="1.905" y2="0" x3="-8.128" y3="22.695" textsize="1.778" layer="51"/>
-<dimension x1="0" y1="43.485" x2="44.43" y2="43.485" x3="22.215" y3="49.276" textsize="1.778" layer="51"/>
-<text x="-5.08" y="9.144" size="0.8128" layer="51" rot="R90">Creepage sample</text>
 <wire x1="42.164" y1="14.732" x2="34.036" y2="14.732" width="1.27" layer="46"/>
 <wire x1="16.637" y1="20.066" x2="11.049" y2="20.066" width="1.27" layer="46"/>
@@
 <wire x1="33.02" y1="31.623" x2="34.29" y2="30.353" width="0.254" layer="1"/>
 <wire x1="34.29" y1="30.353" x2="34.798" y2="30.353" width="0.254" layer="1"/>
+<contactref element="NRF_SMD" pad="CSN"/>
+<wire x1="21.209" y1="38.227" x2="18.643" y2="38.227" width="0.3048" layer="16"/>
+<wire x1="18.643" y1="38.227" x2="18.6424" y2="38.2264" width="0.3048" layer="16"/>
 </signal>
 <signal name="D7">
@@
 </polygon>
 </signal>
-<signal name="N$8">
-<contactref element="NRF_SMD" pad="CSN"/>
-</signal>
 <signal name="N$9">
